Commit message: Updated URDF and MJCF files with measured data and comments

File: workspace/mechanical/FreeCAD/bala2-fire/bala2-fire-simplified.urdf (robot description, URDF)
Before this commit: robot bala2, 3 links, 2 joints
Links:
- link chassis: mass 0.125000 -> 0.127000
Joints:
- joint left_wheel_joint: origin xyz=0 0.0355 0 rpy=0 0 0 -> xyz=0 0.040 0 rpy=0 0 0
- joint right_wheel_joint: origin xyz=0 -0.0355 0 rpy=0 0 0 -> xyz=0 -0.040 0 rpy=0 0 0
